Commit message: finished robot model

File: src/yezibot_description/urdf/yezibot_base.urdf (robot description, URDF)
Before this commit: robot yezibot, 2 links, 1 joints
Links:
- added link imu_link; visual box size=0.02 0.02 0.02
- link base_link: geometry visual cylinder length=0.10 radius=0.2
- link laser_link: geometry visual cylinder length=0.0 radius=0.05
Joints:
- added joint imu_joint: type fixed, parent base_link, child imu_link, origin xyz=0.0 0.0 0.02

Commit message: 差速模型

File: src/yezibot_description/urdf/yezibot_base.urdf (robot description, URDF)
Before this commit: robot yezibot, 3 links, 2 joints
Links:
- removed link base_link
- added link base_footprint
- added link caster_link; visual sphere radius=0.016
- added link left_wheel_link; visual cylinder length=0.04 radius=0.032
- added link right_wheel_link; visual cylinder length=0.04 radius=0.032
Joints:
- added joint base_joint: type fixed, parent base_footprint, child base_link, origin xyz=0.0 0.0 0.076 rpy=0.0 0.0 0.0
- added joint caster_joint: type fixed, parent base_link, child caster_link, origin xyz=0.0 0.0 0.0 rpy=0.06 -0.076 0.0
- added joint left_wheel_joint: type continuous, parent base_link, child left_wheel_link, origin xyz=-0.02 0.10 -0.06 rpy=0 0 0, axis 0 1 0
- added joint right_wheel_joint: type continuous, parent base_link, child right_wheel_link, origin xyz=-0.02 -0.10 -0.06 rpy=0 0 0, axis 0 1 0
- joint laser_joint: origin xyz=0.0 0.0 0.75 -> xyz=0.0 0.0 0.02

Commit message: joint state control

File: src/yezibot_description/urdf/yezibot_base.urdf (robot description, URDF)
Before this commit: robot yezibot, 6 links, 6 joints
Links:
- added link base_link; visual cylinder length=0.12 radius=0.10
